File: 8bc_complete/8bc.kicad_sch (KiCad schematic)
At the start: 1 part, among them J2 Jack-DC

Commit message: updated root
Parts:
- renumbered J2 to J1
Connections:
- no-connect marks 31 -> 0
Other:
- added sheet Instruction Register (8bc_ir.kicad_sch)
