File: 8bc_complete/8bc_clock.kicad_sch (KiCad schematic)
At the start: 25 parts, among them J1 Conn_01x05_Pin, SW1 SW_SPDT, SW2 SW_DIP_x01, U1 ICM7555xP, U2 ICM7555xP, U3 ICM7555xP, U4 74LS04, U5 74LS08, U6 74LS32

Commit message: updated root
Parts:
- renumbered J1 to J2, R4 to R3, R3 to R4, SW2 to SW1, SW1 to SW2, U4 to U2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
