File: 8bc_clock/8bc_clock_4.kicad_pcb (KiCad board)
At the start: 4 copper layers, 61 x 63.5 mm, 27 parts, among them J1 Conn_01x05_Pin, SW1 SW_SPDT, SW2 SW_DIP_x01, U1 ICM7555xP, U2 ICM7555xP, U3 ICM7555xP, U4 74LS04, U5 74LS08, U6 74LS32

Commit message: fixed clock circuit error
Parts:
- removed C1: 0.01uF, Capacitor_THT:C_Disc_D4.7mm_W2.5mm_P5.00mm
- removed C2: 1uF, Capacitor_THT:CP_Radial_D8.0mm_P5.00mm
- removed C3: 0.01uF, Capacitor_THT:C_Radial_D8.0mm_H7.0mm_P3.50mm
- removed C4, C5, C6, C7: 0.1uF, Capacitor_THT:C_Radial_D8.0mm_H7.0mm_P3.50mm
- removed D1: BLUE, LED_THT:LED_D8.0mm
- removed J1: Conn_01x05_Pin, Connector_PinSocket_2.54mm:PinSocket_1x05_P2.54mm_Vertical
- removed R1, R2: 1k, Resistor_THT:R_Axial_DIN0204_L3.6mm_D1.6mm_P7.62mm_Horizontal
- removed R3: 1M, Resistor_THT:R_Axial_DIN0207_L6.3mm_D2.5mm_P7.62mm_Horizontal
- removed R4, R5, R6: 1k, Resistor_THT:R_Axial_DIN0207_L6.3mm_D2.5mm_P7.62mm_Horizontal
- removed R7: 200, Resistor_THT:R_Axial_DIN0207_L6.3mm_D2.5mm_P10.16mm_Horizontal
- removed REF**, REF***: Pin_D1.4mm_L8.5mm_W2.8mm_FlatFork, Connector_Pin:Pin_D1.4mm_L8.5mm_W2.8mm_FlatFork
- removed RV1: R_Potentiometer, Potentiometer_THT:Potentiometer_Alpha_RD901F-40-00D_Single_Vertical
- removed SW1: SW_SPDT, Button_Switch_THT:SW_Slide_1P2T_CK_OS102011MS2Q
- removed SW2: SW_DIP_x01, Button_Switch_THT:SW_PUSH_6mm_H7.3mm
- removed U1, U2, U3: ICM7555xP, Package_DIP:DIP-8_W7.62mm
- removed U4: 74LS04, Package_DIP:DIP-14_W7.62mm
- removed U5: 74LS08, Package_DIP:DIP-14_W7.62mm
- removed U6: 74LS32, Package_DIP:DIP-14_W7.62mm
Routing:
- net Net-(SW1-C): track 79.2 -> 0.00 mm, vias 3 -> 0
- net Net-(U2-TR): track 73.0 -> 0.00 mm, vias 4 -> 0
- net Net-(U3-CV): track 72.6 -> 0.00 mm
- net Net-(U1-THR): track 71.5 -> 0.00 mm
- net Net-(SW1-A): track 69.6 -> 0.00 mm, vias 1 -> 0
- net Net-(U2-DIS): track 65.7 -> 0.00 mm
- net Net-(R2-Pad2): track 58.0 -> 0.00 mm
- net CLK: track 49.7 -> 0.00 mm, vias 1 -> 0
- net Net-(U1-DIS): track 42.6 -> 0.00 mm, vias 2 -> 0
- net HLT: track 41.1 -> 0.00 mm, vias 1 -> 0
- net !CLK: track 40.9 -> 0.00 mm
- net Net-(U2-CV): track 40.6 -> 0.00 mm
- net Net-(U1-CV): track 33.8 -> 0.00 mm, vias 1 -> 0
- net Net-(U3-Q): track 32.6 -> 0.00 mm, vias 1 -> 0
- net Net-(U4-Pad6): track 26.4 -> 0.00 mm
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Other:
- board outline removed
- board text removed: "CLOCK MODULE"
